Commit message: Add Dockerfile and entrypoint script; rename barracuda.xacro with updated mesh reference

File: catkin_ws/barracuda_description/urdf/barracuda.xacro (robot description, xacro)
@@ -17,5 +17,5 @@
             <origin xyz="0 0 -0.9" rpy="0 0 1.5708"/>
             <geometry>
-                <mesh filename="file://$(find barracuda_description)/meshes/virgil.dae" scale="1 1 1"/>
+                <mesh filename="file://$(find barracuda_description)/meshes/mantaray_base_link.stl" scale="1 1 1"/>
             </geometry>
         </visual>
@@ -23,5 +23,5 @@
             <origin xyz="0 0 -0.9" rpy="0 0 1.5708"/>
             <geometry>
-                <mesh filename="file://$(find barracuda_description)/meshes/virgil.dae" scale="1 1 1"/>
+                <mesh filename="file://$(find barracuda_description)/meshes/mantaray_base_link.stl" scale="1 1 1"/>
             </geometry>
         </collision>
